File: Rev1.kicad_pcb (KiCad board)
At the start: 2 copper layers, 152.8 x 71.5 mm, 105 parts, among them J1 Conn_01x08_Socket, J10 Conn_01x08_Socket, J11 Conn_01x02_Socket, J12 Conn_01x08_Socket, J13 Conn_01x08_Socket, J2 Conn_01x08_Socket, J3 Conn_01x08_Socket, J4 Conn_01x08_Socket, J5 Conn_01x08_Socket, J6 Conn_01x08_Socket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

Commit message: Update, pics
Parts:
- J11: value Conn_01x02_Socket -> Power
Changed lines of the file:
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@@
 			)
 		)
-		(property "Value" "Conn_01x02_Socket"
-			(at 0 2.965001 90)
-			(layer "F.Fab")
+		(property "Value" "Power"
+			(at 2.1336 0.770392 180)
+			(layer "F.SilkS")
 			(effects
 				(font
@@
 		)
 		(fp_text user "${REFERENCE}"
-			(at 0 0.635 360)
+			(at 0 0.635 0)
 			(layer "F.Fab")
 			(effects
@@
 		)
 		(fp_text user "${REFERENCE}"
-			(at 0 4.445001 360)
+			(at 0 4.445001 0)
 			(layer "F.Fab")
 			(effects
@@
 		(polygon
 			(pts
-				(xy 103.2256 22.098) (xy 257.2004 22.098) (xy 257.2004 96.4692) (xy 257.2004 96.4692) (xy 103.2256 96.4692)
+				(xy 103.2256 22.098) (xy 257.2004 22.098) (xy 257.2004 96.4692) (xy 103.2256 96.4692)
 			)
 		)
